Commit message: Ver 1.2 Car Spec Update & key_teleop Update

File: simulate_ws/src/server/urdf/car.xacro (robot description, xacro)
@@ -2,9 +2,7 @@
 <robot name="erp42" xmlns:xacro="http://www.ros.org/wiki/xacro">
     <xacro:arg name="car_name" default="car1"/>
-    <xacro:property name="mass" value="10.0"/>
-    <xacro:property name="wheelbase" value="0.3"/>
-    <xacro:property name="track_width" value="0.2"/>
-    <xacro:property name="wheel_radius" value="0.05"/>
-    <xacro:property name="wheel_mass" value="1.0"/>
+    <xacro:property name="mass" value="200.0"/>
+    <xacro:property name="wheelbase" value="1.0"/>
+    <xacro:property name="wheel_mass" value="5.0"/>
     <link name="$(arg car_name)/chassis">
         <visual>
@@ -248,5 +246,5 @@
             <wheel_separation>0.2</wheel_separation>
             <wheel_radius>0.27</wheel_radius>
-            <steering_limit>0.6</steering_limit>
+            <steering_limit>0.3491</steering_limit>
             <odom_publish_frequency>50.0</odom_publish_frequency>
             <topic>/$(arg car_name)/cmd_vel</topic>
@@ -271,15 +269,15 @@
             <update_rate>20.0</update_rate>
             <topic>/$(arg car_name)/scan</topic>
-            <gz_frame_id>$(arg car_name)</gz_frame_id>
+            <gz_frame_id>$(arg car_name)/lidar_link</gz_frame_id>
             <lidar>
                 <scan>
                     <horizontal>
-                        <samples>360</samples>
-                        <resolution>0.1</resolution>
+                        <samples>1800</samples>
+                        <resolution>1.0</resolution>
                         <min_angle>-3.14159</min_angle>
                         <max_angle>3.14159</max_angle>
                     </horizontal>
                     <vertical>
-                        <samples>30</samples>
+                        <samples>16</samples>
                         <resolution>1.0</resolution>
                         <min_angle>-0.2618</min_angle>
@@ -288,7 +286,7 @@
                 </scan>
                 <range>
-                    <min>0.3</min>
+                    <min>0.5</min>
                     <max>100.0</max>
-                    <resolution>0.1</resolution>
+                    <resolution>0.002</resolution>
                 </range>
             </lidar>
@@ -301,5 +299,5 @@
             <update_rate>20.0</update_rate>
             <topic>/$(arg car_name)/camera/image_raw</topic>
-            <gz_frame_id>$(arg car_name)</gz_frame_id>
+            <gz_frame_id>$(arg car_name)/camera_link</gz_frame_id>
             <camera>
                 <horizontal_fov>1.047</horizontal_fov>
@@ -322,5 +320,5 @@
             <update_rate>10.0</update_rate>
             <topic>/$(arg car_name)/gps/fix</topic>
-            <gz_frame_id>$(arg car_name)</gz_frame_id>
+            <gz_frame_id>$(arg car_name)/gps_link</gz_frame_id>
             <navsat>
                 <position_sensing>

File: simulate_ws/src/server/urdf/test.xacro (robot description, xacro)
@@ -11,5 +11,5 @@
             <origin xyz="0.0 0.0 0.0" rpy="0.0 0.0 0.0"/>
             <geometry>
-                <mesh filename="/home/th/simulate_ws/src/server/mesh/body.stl" scale="1.0 1.0 1.0"/>
+                <mesh filename="/home/th/Autonomous-Racing-Simulator/simulate_ws/src/server/mesh/body.stl" scale="1.0 1.0 1.0"/>
             </geometry>
             <material name="whiteblue">
@@ -20,5 +20,5 @@
             <origin xyz="0.0 0.0 0.0" rpy="0.0 0.0 0.0"/>
             <geometry>
-                <mesh filename="/home/th/simulate_ws/src/server/mesh/body.stl" scale="1.0 1.0 1.0"/>
+                <mesh filename="/home/th/Autonomous-Racing-Simulator/simulate_ws/src/server/mesh/body.stl" scale="1.0 1.0 1.0"/>
             </geometry>
         </collision>
@@ -33,5 +33,5 @@
             <origin xyz="0.0 0.0 0.0" rpy="0.0 0.0 0.0"/>
             <geometry>
-                <mesh filename="/home/th/simulate_ws/src/server/mesh/left.stl" scale="1.0 1.0 1.0"/>
+                <mesh filename="/home/th/Autonomous-Racing-Simulator/simulate_ws/src/server/mesh/left.stl" scale="1.0 1.0 1.0"/>
             </geometry>
             <material name="black">
@@ -55,5 +55,5 @@
             <origin xyz="0.0 0.0 0.0" rpy="0.0 0.0 0.0"/>
             <geometry>
-                <mesh filename="/home/th/simulate_ws/src/server/mesh/right.stl" scale="1.0 1.0 1.0"/>
+                <mesh filename="/home/th/Autonomous-Racing-Simulator/simulate_ws/src/server/mesh/right.stl" scale="1.0 1.0 1.0"/>
             </geometry>
             <material name="black">
@@ -77,5 +77,5 @@
             <origin xyz="0.0 0.0 0.0" rpy="0.0 0.0 0.0"/>
             <geometry>
-                <mesh filename="/home/th/simulate_ws/src/server/mesh/left.stl" scale="1.0 1.0 1.0"/>
+                <mesh filename="/home/th/Autonomous-Racing-Simulator/simulate_ws/src/server/mesh/left.stl" scale="1.0 1.0 1.0"/>
             </geometry>
             <material name="black">
@@ -99,5 +99,5 @@
             <origin xyz="0.0 0.0 0.0" rpy="0.0 0.0 0.0"/>
             <geometry>
-                <mesh filename="/home/th/simulate_ws/src/server/mesh/right.stl" scale="1.0 1.0 1.0"/>
+                <mesh filename="/home/th/Autonomous-Racing-Simulator/simulate_ws/src/server/mesh/right.stl" scale="1.0 1.0 1.0"/>
             </geometry>
             <material name="black">

Commit message: Ver 1.3 Add Livox Lidar

File: simulate_ws/src/server/urdf/car.xacro (robot description, xacro)
@@ -184,4 +184,30 @@
         <child link="$(arg car_name)/lidar_link"/>
         <origin xyz="-0.3 0.0 0.95" rpy="0.0 0.0 0.0"/>
+    </joint>
+    <link name="$(arg car_name)/livox_lidar_link">
+        <visual>
+            <origin xyz="0.0 0.0 0.0" rpy="0.0 0.0 0.0"/>
+            <geometry>
+                <box size="0.115 0.077 0.0841"/>
+            </geometry>
+            <material name="Gray">
+                <color rgba="0.169 0.169 0.169 1"/>
+            </material>
+        </visual>
+        <collision>
+            <origin xyz="0.0 0.0 0.0" rpy="0.0 0.0 0.0"/>
+            <geometry>
+                <box size="0.115 0.077 0.0841"/>
+            </geometry>
+        </collision>
+        <inertial>
+            <mass value="1.18"/>
+            <inertia ixx="0.001" ixy="0.0" ixz="0.0" iyy="0.001" iyz="0.0" izz="0.001"/>
+        </inertial>
+    </link>
+    <joint name="$(arg car_name)/livox_lidar_joint" type="fixed">
+        <parent link="$(arg car_name)/chassis"/>
+        <child link="$(arg car_name)/livox_lidar_link"/>
+        <origin xyz="0.055 0.0 0.74" rpy="0.0 0.0524 0.0"/>
     </joint>
     <link name="$(arg car_name)/camera_link">
@@ -264,5 +290,5 @@
     </gazebo>
     <gazebo reference="$(arg car_name)/lidar_link">
-        <sensor name="gpu_lidar" type="gpu_lidar">
+        <sensor name="velodyne_lidar" type="gpu_lidar">
             <always_on>true</always_on>
             <visualize>false</visualize>
@@ -293,4 +319,34 @@
         </sensor>
     </gazebo>
+    <gazebo reference="$(arg car_name)/livox_lidar_link">
+        <sensor name="livox_lidar" type="gpu_lidar">
+            <always_on>true</always_on>
+            <visualize>false</visualize>
+            <update_rate>10.0</update_rate>
+            <topic>/$(arg car_name)/livox</topic>
+            <gz_frame_id>$(arg car_name)/livox_lidar_link</gz_frame_id>
+            <lidar>
+                <scan>
+                    <horizontal>
+                        <samples>400</samples>
+                        <resolution>1.0</resolution>
+                        <min_angle>-0.713</min_angle>
+                        <max_angle>0.713</max_angle>
+                    </horizontal>
+                    <vertical>
+                        <samples>120</samples>
+                        <resolution>1.0</resolution>
+                        <min_angle>-0.219</min_angle>
+                        <max_angle>0.219</max_angle>
+                    </vertical>
+                </scan>
+                <range>
+                    <min>0.5</min>
+                    <max>260.0</max>
+                    <resolution>0.002</resolution>
+                </range>
+            </lidar>
+        </sensor>
+    </gazebo>
     <gazebo reference="$(arg car_name)/camera_link">
         <sensor name="camera" type="camera">

File: simulate_ws/src/server/urdf/test.xacro (robot description, xacro)
@@ -123,25 +123,4 @@
         <inertial><mass value="0.1"/><inertia ixx="0.001" ixy="0.0" ixz="0.0" iyy="0.001" iyz="0.0" izz="0.001"/></inertial>
     </link>
-    <link name="lidar_link">
-        <visual>
-            <origin xyz="0.0 0.0 0.0" rpy="0.0 0.0 0.0"/>
-            <geometry>
-                <cylinder radius="0.05165" length="0.0717"/>
-            </geometry>
-            <material name="Gray">
-                <color rgba="0.169 0.169 0.169 1"/>
-            </material>
-        </visual>
-        <collision>
-            <origin xyz="0.0 0.0 0.0" rpy="0.0 0.0 0.0"/>
-            <geometry>
-                <cylinder radius="0.05165" length="0.0717"/>
-            </geometry>
-        </collision>
-        <inertial>
-            <mass value="0.83"/>
-            <inertia ixx="0.001" ixy="0.0" ixz="0.0" iyy="0.001" iyz="0.0" izz="0.001"/>
-        </inertial>
-    </link>
     <joint name="rear_left_joint" type="continuous">
         <parent link="chassis"/>
@@ -182,8 +161,55 @@
         <axis xyz= "0 1 0"/>
     </joint>
+    <link name="lidar_link">
+        <visual>
+            <origin xyz="0.0 0.0 0.0" rpy="0.0 0.0 0.0"/>
+            <geometry>
+                <cylinder radius="0.05165" length="0.0717"/>
+            </geometry>
+            <material name="Gray">
+                <color rgba="0.169 0.169 0.169 1"/>
+            </material>
+        </visual>
+        <collision>
+            <origin xyz="0.0 0.0 0.0" rpy="0.0 0.0 0.0"/>
+            <geometry>
+                <cylinder radius="0.05165" length="0.0717"/>
+            </geometry>
+        </collision>
+        <inertial>
+            <mass value="0.83"/>
+            <inertia ixx="0.001" ixy="0.0" ixz="0.0" iyy="0.001" iyz="0.0" izz="0.001"/>
+        </inertial>
+    </link>
     <joint name="lidar_joint" type="fixed">
         <parent link="chassis"/>
         <child link="lidar_link"/>
         <origin xyz="-0.3 0.0 0.95" rpy="0.0 0.0 0.0"/>
+    </joint>
+    <link name="livox_lidar_link">
+        <visual>
+            <origin xyz="0.0 0.0 0.0" rpy="0.0 0.0 0.0"/>
+            <geometry>
+                <box size="0.115 0.077 0.0841"/>
+            </geometry>
+            <material name="Gray">
+                <color rgba="0.169 0.169 0.169 1"/>
+            </material>
+        </visual>
+        <collision>
+            <origin xyz="0.0 0.0 0.0" rpy="0.0 0.0 0.0"/>
+            <geometry>
+                <box size="0.115 0.077 0.0841"/>
+            </geometry>
+        </collision>
+        <inertial>
+            <mass value="1.18"/>
+            <inertia ixx="0.001" ixy="0.0" ixz="0.0" iyy="0.001" iyz="0.0" izz="0.001"/>
+        </inertial>
+    </link>
+    <joint name="livox_lidar_joint" type="fixed">
+        <parent link="chassis"/>
+        <child link="livox_lidar_link"/>
+        <origin xyz="0.055 0.0 0.74" rpy="0.0 0.0524 0.0"/>
     </joint>
     <link name="camera_link">
